File: hardware/v2/pdlc-output.kicad_sch (KiCad schematic)
At the start: 16 parts, among them U6 LMR38010SDDAR

Commit message: WIP
Parts:
- removed D1: SMAJ78A, Diode_SMD:D_SMA, symbol Diode:SMAJ78A
- removed R21: 10K, Resistor_SMD:R_0402_1005Metric, symbol Device:R
- added D8: SMF70A, Diode_SMD:D_SMF, symbol Diode:SMF16A
- added R39: 22K, Resistor_SMD:R_0402_1005Metric, symbol Device:R
- C30: renamed from C31; Alternative GCM32DC72A475KE02L -> (none); MPN HMK325C7475KN-TE -> (none); Part (none) -> HMK325C7475KN-TE; Part Alternative (none) -> GCM32DC72A475KE02L
- C31: renamed from C28; MPN CL31B104KCFNNNE -> (none); Part (none) -> CL31B104KCFNNNE
- C34: renamed from C25; MPN CL31B104KCFNNNE -> (none); Part (none) -> CL31B104KCFNNNE
- C35: renamed from C29; MPN GRM32EC72A106KE05L -> (none); Part (none) -> GRM32EC72A106KE05L
- C36: renamed from C30; MPN GRM32EC72A106KE05L -> (none); Part (none) -> GRM32EC72A106KE05L
- L2: FT Rotation Offset (none) -> 270; MPN 7447714680 -> (none); Part (none) -> 7447714680
- renumbered C27 to C32, C26 to C33, R15 to R34, R3 to R35, R13 to R36, R12 to R37, R14 to R38
Connections:
- net +3.3V: now also R39.1
- net GND: now also D8.2 (A2)
- net PG: now also R39.2
- net VOUT: now also D8.1 (A1)
