File: hardware/v2/pdlc-output.kicad_sch (KiCad schematic)
At the start: 16 parts, among them U6 LMR38010SDDAR

Commit message: WIP
Parts:
- R35: renamed from R21; Rating 50V, 1% -> 50V
- renumbered C31 to C30, C28 to C31, C27 to C32, C26 to C33, C25 to C34, C29 to C35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
