File: hardware/v2/pdlc.kicad_pcb (KiCad board)
At the start: 4 copper layers, 21 parts

Commit message: Finalize for production of v2 revision.
Parts:
- removed REF**: TSOT-23-5, Package_TO_SOT_SMD:TSOT-23-5
- removed REF**: CP_Elec_6.3x9.9, Capacitor_SMD:CP_Elec_6.3x9.9
- removed REF**: CP_Radial_D8.0mm_P3.50mm, Capacitor_THT:CP_Radial_D8.0mm_P3.50mm
- removed REF**: C_2220_5750Metric, Capacitor_SMD:C_2220_5750Metric
- removed REF**: D_SMF, Diode_SMD:D_SMF
- removed REF**: CP_Elec_10x12.6, Capacitor_SMD:CP_Elec_10x12.6
- removed REF**: SC-74A-5_1.55x2.9mm_P0.95mm, Package_TO_SOT_SMD:SC-74A-5_1.55x2.9mm_P0.95mm
- removed REF**: D_SMB, Diode_SMD:D_SMB
- removed REF**: C_1206_3216Metric, Capacitor_SMD:C_1206_3216Metric
- removed REF**: SOT-23, Package_TO_SOT_SMD:SOT-23
- removed REF**: D_SOD-323, Diode_SMD:D_SOD-323
- removed REF**: D_SMA, Diode_SMD:D_SMA
- removed REF**: SOT-323_SC-70, Package_TO_SOT_SMD:SOT-323_SC-70
- removed REF**: C_1812_4532Metric, Capacitor_SMD:C_1812_4532Metric
- removed REF** (x2): C_1210_3225Metric, Capacitor_SMD:C_1210_3225Metric
- removed REF** (x2): D_SMC, Diode_SMD:D_SMC
- removed REF**: D_SOD-123, Diode_SMD:D_SOD-123
- removed REF**: CP_Radial_D6.3mm_P2.50mm, Capacitor_THT:CP_Radial_D6.3mm_P2.50mm
- removed REF**: SOT-23-5_HandSoldering, Package_TO_SOT_SMD:SOT-23-5_HandSoldering
- added C1: 100n, Capacitor_SMD:C_0402_1005Metric, F.Cu at (149.0, 76.8)
- added C10: 100n, Capacitor_SMD:C_0603_1608Metric, F.Cu at (93.5, 94.2)
- added C11: 1u, Capacitor_SMD:C_0805_2012Metric, F.Cu at (93.2, 90.8)
- added C12: 100n, Capacitor_SMD:C_1206_3216Metric, F.Cu at (110.0, 89.8)
- added C13: 4.7u, Capacitor_SMD:C_1210_3225Metric, F.Cu at (107.5, 85.2)
- added C14: 4.7u, Capacitor_SMD:C_1210_3225Metric, F.Cu at (112.8, 85.2)
- added C15: 22u, Capacitor_SMD:CP_Elec_6.3x9.9, F.Cu at (110.0, 79.2)
- added C16: 220n, Capacitor_SMD:C_0402_1005Metric, F.Cu at (102.0, 96.5)
- added C17: 2.2n, Capacitor_SMD:C_0603_1608Metric, F.Cu at (98.5, 95.0)
- added C18: 22n, Capacitor_SMD:C_0402_1005Metric, F.Cu at (100.0, 96.5)
- added C19: 10u, Capacitor_SMD:C_0603_1608Metric, F.Cu at (140.5, 88.5)
- added C2: 100n, Capacitor_SMD:C_0402_1005Metric, F.Cu at (145.5, 76.8)
- added C20: 100n, Capacitor_SMD:C_0402_1005Metric, F.Cu at (130.5, 88.5)
- added C21: 100n, Capacitor_SMD:C_0402_1005Metric, F.Cu at (138.1, 99.6)
- added C22: 100n, Capacitor_SMD:C_0402_1005Metric, F.Cu at (141.5, 90.8)
- added C23: 100n, Capacitor_SMD:C_0402_1005Metric, F.Cu at (132.4, 87.2)
- added C24: 1u, Capacitor_SMD:C_0603_1608Metric, F.Cu at (127.2, 93.8)
- added C25: 100n, Capacitor_SMD:C_0402_1005Metric, F.Cu at (129.0, 94.2)
- added C26: 100n, Capacitor_SMD:C_0402_1005Metric, F.Cu at (129.0, 91.2)
- added C27: 100n, Capacitor_SMD:C_0402_1005Metric, F.Cu at (142.8, 104.8)
- added C28: 100n, Capacitor_SMD:C_0402_1005Metric, F.Cu at (142.8, 120.8)
- added C29: 100n, Capacitor_SMD:C_0402_1005Metric, F.Cu at (142.8, 114.2)
- added C3: 1u, Capacitor_SMD:C_0805_2012Metric, F.Cu at (118.2, 84.0)
- added C30: 4.7u, Capacitor_SMD:C_1210_3225Metric, F.Cu at (117.0, 107.2)
- added C31: 100n, Capacitor_SMD:C_1206_3216Metric, F.Cu at (113.8, 107.2)
- added C32: 100n, Capacitor_SMD:C_0603_1608Metric, F.Cu at (107.8, 100.2)
- added C33: C, Capacitor_SMD:C_0603_1608Metric, F.Cu at (115.0, 103.0)
- added C34: 100n, Capacitor_SMD:C_1206_3216Metric, F.Cu at (88.0, 107.0)
- added C35: 10u, Capacitor_SMD:C_1210_3225Metric, F.Cu at (91.2, 101.5)
- added C36: 10u, Capacitor_SMD:C_1210_3225Metric, F.Cu at (91.2, 107.0)
- added C37: 4.7u, Capacitor_SMD:C_1210_3225Metric, F.Cu at (117.0, 120.8)
- added C38: 100n, Capacitor_SMD:C_1206_3216Metric, F.Cu at (113.8, 120.8)
- added C39: 100n, Capacitor_SMD:C_0603_1608Metric, F.Cu at (107.8, 113.8)
- added C4: 10n, Capacitor_SMD:C_0402_1005Metric, F.Cu at (119.0, 89.8)
- added C40: C, Capacitor_SMD:C_0603_1608Metric, F.Cu at (115.0, 116.5)
- added C41: 100n, Capacitor_SMD:C_1206_3216Metric, F.Cu at (88.0, 120.5)
- added C42: 10u, Capacitor_SMD:C_1210_3225Metric, F.Cu at (91.2, 115.0)
- added C43: 10u, Capacitor_SMD:C_1210_3225Metric, F.Cu at (91.2, 120.5)
- added C5: 2.2u, Capacitor_SMD:C_0603_1608Metric, F.Cu at (122.0, 87.2)
- added C6: 220u, Capacitor_THT:CP_Radial_D6.3mm_P2.50mm, F.Cu at (89.6, 79.9)
- added C7: 10u, Capacitor_SMD:C_1210_3225Metric, F.Cu at (89.2, 85.5)
- added C8: 10u, Capacitor_SMD:C_1210_3225Metric, F.Cu at (89.2, 89.2)
- added C9: 10u, Capacitor_SMD:C_1210_3225Metric, F.Cu at (89.2, 93.0)
- added D1: SMF16A, Diode_SMD:D_SMF, F.Cu at (83.2, 85.2)
- added D2: B2100-13-F, Diode_SMD:D_SMB, F.Cu at (104.0, 90.8)
- added D3: PESD3V3L5UY, Package_TO_SOT_SMD:SOT-363_SC-70-6, F.Cu at (129.2, 114.5)
- added D4: PESD3V3L5UY, Package_TO_SOT_SMD:SOT-363_SC-70-6, F.Cu at (134.2, 114.5)
- added D5: LTST-C19HE1WT, LED_SMD:LED_LiteOn_LTST-C19HE1WT, F.Cu at (147.0, 95.0)
- added D6: KT-0603R, LED_SMD:LED_0603_1608Metric, F.Cu at (147.0, 86.5)
- added D7: 1N5819WS, Diode_SMD:D_SOD-323, F.Cu at (149.0, 110.8)
- added D8: SMF70A, Diode_SMD:D_SMF, F.Cu at (88.0, 101.5)
- added D9: SMF70A, Diode_SMD:D_SMF, F.Cu at (88.0, 115.0)
- added F1: 1812L200/16DR, 1812L:1812L, F.Cu at (78.5, 84.8)
- added FB1: 450mOhm, Inductor_SMD:L_0603_1608Metric, F.Cu at (128.0, 96.2)
- added J1: SM04B-SRSS-TB, Connector_JST:JST_SH_SM04B-SRSS-TB_1x04-1MP_P1.00mm_Horizontal, F.Cu at (156.5, 79.5)
- added J2: TBP04R12-500-04BE, Connector_Phoenix_MSTB:PhoenixContact_MSTBA_2,5_4-G_1x04_P5.00mm_Horizontal, F.Cu at (82.5, 92.5)
- added J3: SM04B-SRSS-TB, Connector_JST:JST_SH_SM04B-SRSS-TB_1x04-1MP_P1.00mm_Horizontal, F.Cu at (156.5, 87.8)
- added J4: Conn_02x08_Odd_Even, Connector_PinSocket_2.54mm:PinSocket_2x08_P2.54mm_Vertical, F.Cu at (138.8, 80.2)
- added J5: Conn_ST_STDC14, Samtec:SAMTEC_FTSH-107-01-L-DV-K-A, F.Cu at (131.2, 121.0)
- added J6: TBP03R1-350-06BE, Connector_Phoenix_MC:PhoenixContact_MC_1,5_6-G-3.5_1x06_P3.50mm_Horizontal, F.Cu at (154.3, 121.4)
- added JP1: SolderJumper_2_Open, Jumper:SolderJumper-2_P1.3mm_Open_TrianglePad1.0x1.5mm, F.Cu at (147.0, 122.0)
- added L1: 15u, WE-PD_1050P:WE-PD_1050P, F.Cu at (98.5, 82.5)
- added L2: 68u, WE-PD_1050P:WE-PD_1050P, F.Cu at (99.5, 104.2)
- added L3: 68u, WE-PD_1050P:WE-PD_1050P, F.Cu at (99.5, 117.8)
- added MP1: MountingHole_2.7mm_M2.5, MountingHole:MountingHole_2.7mm_M2.5, F.Cu at (78.5, 78.5)
- added MP1: MountingHole_2.7mm_M2.5, MountingHole:MountingHole_2.7mm_M2.5, F.Cu at (78.5, 121.5)
- added MP1: MountingHole_2.7mm_M2.5, MountingHole:MountingHole_2.7mm_M2.5, F.Cu at (149.0, 100.0)
- added Q1: 2N7002, Package_TO_SOT_SMD:SOT-23, F.Cu at (116.2, 94.5)
- added Q2: MMBT3904, Package_TO_SOT_SMD:SOT-23, F.Cu at (111.2, 94.5)
- added Q3: 2N7002, Package_TO_SOT_SMD:SOT-23, F.Cu at (146.0, 110.8)
- added R1: 2.2K, Resistor_SMD:R_0402_1005Metric, F.Cu at (142.8, 79.0)
- added R10: 37.4K, Resistor_SMD:R_0402_1005Metric, F.Cu at (105.5, 96.5)
- added R11: 13K, Resistor_SMD:R_0402_1005Metric, F.Cu at (95.5, 94.8)
- added R12: 470, Resistor_SMD:R_0402_1005Metric, F.Cu at (119.2, 95.0)
- added R13: 15K, Resistor_SMD:R_0402_1005Metric, F.Cu at (90.5, 96.8)
- added R14: 100K, Resistor_SMD:R_0402_1005Metric, F.Cu at (119.2, 92.8)
- added R15: 2.2K, Resistor_SMD:R_0402_1005Metric, F.Cu at (136.8, 83.5)
- added R16: 2.2K, Resistor_SMD:R_0402_1005Metric, F.Cu at (138.8, 83.5)
- added R17: 10K, Resistor_SMD:R_0402_1005Metric, F.Cu at (132.2, 85.0)
- added R18: 10K, Resistor_SMD:R_0402_1005Metric, F.Cu at (140.5, 98.2)
- added R19: 10K, Resistor_SMD:R_0402_1005Metric, F.Cu at (128.0, 85.0)
- added R2: 2.2K, Resistor_SMD:R_0402_1005Metric, F.Cu at (141.5, 79.0)
- added R20: 100K, Resistor_SMD:R_0402_1005Metric, F.Cu at (136.8, 122.5)
- added R21: 100K, Resistor_SMD:R_0402_1005Metric, F.Cu at (136.8, 119.0)
- added R22: 1K, Resistor_SMD:R_0402_1005Metric, F.Cu at (147.0, 93.0)
- added R23: 22K, Resistor_SMD:R_0402_1005Metric, F.Cu at (142.8, 107.2)
- added R24: 22K, Resistor_SMD:R_0402_1005Metric, F.Cu at (142.8, 123.2)
- added R25: 470, Resistor_SMD:R_0402_1005Metric, F.Cu at (147.0, 91.8)
- added R26: 470, Resistor_SMD:R_0402_1005Metric, F.Cu at (147.0, 90.5)
- added R27: 2.2K, Resistor_SMD:R_0402_1005Metric, F.Cu at (142.8, 106.0)
- added R28: 2.2K, Resistor_SMD:R_0402_1005Metric, F.Cu at (142.8, 122.0)
- added R29: 1K, Resistor_SMD:R_0402_1005Metric, F.Cu at (147.0, 88.2)
- added R3: 330K, Resistor_SMD:R_0603_1608Metric, F.Cu at (105.0, 95.0)
- added R30: 22K, Resistor_SMD:R_0402_1005Metric, F.Cu at (142.8, 116.8)
- added R31: 2.2K, Resistor_SMD:R_0402_1005Metric, F.Cu at (142.8, 115.5)
- added R32: 470, Resistor_SMD:R_0402_1005Metric, F.Cu at (142.8, 111.8)
- added R33: 100K, Resistor_SMD:R_0402_1005Metric, F.Cu at (142.8, 110.5)
- added R34: 220K, Resistor_SMD:R_0603_1608Metric, F.Cu at (113.2, 103.0)
- added R35: 1M, Resistor_SMD:R_0805_2012Metric, F.Cu at (78.5, 115.2)
- added R36: 4.7K, Resistor_SMD:R_0603_1608Metric, F.Cu at (112.2, 100.2)
- added R37: 10K, Resistor_SMD:R_0603_1608Metric, F.Cu at (115.8, 100.2)
- added R38: 51K, Resistor_SMD:R_0402_1005Metric, F.Cu at (118.0, 103.5)
- added R39: 22K, Resistor_SMD:R_0402_1005Metric, F.Cu at (127.5, 99.2)
- added R4: 5.1K, Resistor_SMD:R_0603_1608Metric, F.Cu at (101.8, 95.0)
- added R40: 220K, Resistor_SMD:R_0603_1608Metric, F.Cu at (113.2, 116.5)
- added R41: 1M, Resistor_SMD:R_0805_2012Metric, F.Cu at (83.5, 115.2)
- added R42: 4.7K, Resistor_SMD:R_0603_1608Metric, F.Cu at (112.2, 113.8)
- added R43: 10K, Resistor_SMD:R_0603_1608Metric, F.Cu at (115.8, 113.8)
- added R44: 51K, Resistor_SMD:R_0402_1005Metric, F.Cu at (118.0, 117.0)
- added R45: 22K, Resistor_SMD:R_0402_1005Metric, F.Cu at (127.5, 97.8)
- added R5: 22K, Resistor_SMD:R_0402_1005Metric, F.Cu at (121.2, 92.0)
- added R6: 22K, Resistor_SMD:R_0402_1005Metric, F.Cu at (124.0, 93.8)
- added R7: 100K, Resistor_SMD:R_0402_1005Metric, F.Cu at (114.2, 92.2)
- added R8: 100K, Resistor_SMD:R_0402_1005Metric, F.Cu at (90.5, 95.5)
- added R9: 1K, Resistor_SMD:R_0402_1005Metric, F.Cu at (98.0, 96.5)
- added SW1: SW_Push, Button_Switch_SMD:SW_SPST_TS-1088-xR020, F.Cu at (147.0, 106.0)
- added SW2: SW_Push, Button_Switch_SMD:SW_SPST_TS-1088-xR020, F.Cu at (147.0, 115.5)
- added TH1: JLCPCB_PCBA_Tooling_Hole, Generic:JLCPCB_PCBA_Tooling_Hole, F.Cu at (83.0, 77.0)
- added TH1: JLCPCB_PCBA_Tooling_Hole, Generic:JLCPCB_PCBA_Tooling_Hole, F.Cu at (83.0, 123.0)
- added TH1: JLCPCB_PCBA_Tooling_Hole, Generic:JLCPCB_PCBA_Tooling_Hole, F.Cu at (158.0, 119.6)
- added U1: LP2985-33DBVR, Package_TO_SOT_SMD:SOT-23-5, F.Cu at (118.5, 87.2)
- added U2: ISO1640, Package_SO:SOIC-8_3.9x4.9mm_P1.27mm, F.Cu at (147.2, 80.2)
- added U3: SN74LVC1G08DCKR, Package_TO_SOT_SMD:SOT-353_SC-70-5, F.Cu at (121.8, 94.5)
- added U4: LM5158, LM5158:LM5158, F.Cu at (97.0, 91.5)
- added U5: STM32L151C8T6A, Package_QFP:LQFP-48_7x7mm_P0.5mm, F.Cu at (135.2, 93.5)
- added U6: LMR38010SDDAR, Package_SO:TI_SO-PowerPAD-8, F.Cu at (109.0, 105.5)
- added U7: LMR38010SDDAR, Package_SO:TI_SO-PowerPAD-8, F.Cu at (109.0, 119.0)
Routing:
- net +12V: track 0.00 -> 161.1 mm, vias 0 -> 2
- net /HV: track 0.00 -> 86.3 mm
- net /PDLC_EN_DRV: track 0.00 -> 62.3 mm, vias 0 -> 2
- net GND: track 0.00 -> 62.0 mm, vias 0 -> 322
- net /HV_PG: track 0.00 -> 53.2 mm, vias 0 -> 4
- net /PDLC_OUT_A: track 0.00 -> 50.8 mm, vias 0 -> 2
- net /~{RESET}: track 0.00 -> 47.4 mm, vias 0 -> 2
- net /PDLC_OUT_B: track 0.00 -> 44.4 mm, vias 0 -> 2
- net /PDLC_PG_B: track 0.00 -> 43.4 mm, vias 0 -> 4
- net +3.3V: track 0.00 -> 41.8 mm, vias 0 -> 25
- net /CONSOLE_RX: track 0.00 -> 39.4 mm, vias 0 -> 2
- net /SWO: track 0.00 -> 37.1 mm, vias 0 -> 2
- net /SWCLK: track 0.00 -> 36.6 mm, vias 0 -> 2
- net /INT_I2C_SCL: track 0.00 -> 36.4 mm
- net /SWDIO: track 0.00 -> 35.9 mm, vias 0 -> 2
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- added copper zone on In2.Cu, net +3.3V
- added copper zone on F.Cu, net /BUS_GND
- added copper zone on In1.Cu, net /BUS_GND
- added copper zone on B.Cu, net GND
- added copper zone on F.Cu, net GND
- added copper zone on In1.Cu, net GND
- added copper zone on In2.Cu, net GND
Other:
- board outline added: 85 x 50 mm
- board text added: "${COMPANY} ${TITLE} ${ISSUE_DATE}, ${REVISION} github.com/ brown-studios/pdlc"
- board text added: "1: GND 2: 12V_IN 3: PDLC_OUT_A 4: PDLC_OUT_B"
- board text added: "1: GND 2: 3.3V 3: SDA 4: SCL"
- board text added: "6: 12V_OUT 5: LOAD_OUT 4: GND 3: CTRL_MODE_IN 2: CTRL_EN_IN 1: GND"
- board text added: "BT0 PC13 PB6 PB15 PB13 SCL2 3V3 12V"
- board text added: "CONTROL"
- board text added: "DEBUG"
- board text added: "EN"
- board text added: "EXPANSION"
- board text added: "EXT I2C"
- board text added: "MODE"
- board text added: "POWER"
- board text added: "RST PA3 PB7 PA15 PB14 SDA2 GND GND"
- board text added: "SET"
- board text added: "STATUS"
