File: hardware/v2/pdlc.kicad_pcb (KiCad board)
At the start: 4 copper layers, 21 parts

Commit message: WIP
Parts:
- added REF**: PhoenixContact_MSTBA_2,5_4-G_1x04_P5.00mm_Horizontal, Connector_Phoenix_MSTB:PhoenixContact_MSTBA_2,5_4-G_1x04_P5.00mm_Horizontal, F.Cu at (31.4, 41.3)
- added REF**: D_SMA, Diode_SMD:D_SMA, F.Cu at (77.8, 89.1)
- added REF**: PhoenixContact_MC_1,5_4-G-3.5_1x04_P3.50mm_Horizontal, Connector_Phoenix_MC:PhoenixContact_MC_1,5_4-G-3.5_1x04_P3.50mm_Horizontal, F.Cu at (45.8, 72.9)
- added REF**: D_SOD-123, Diode_SMD:D_SOD-123, F.Cu at (94.8, 74.1)
- added REF**: D_SOD-323, Diode_SMD:D_SOD-323, F.Cu at (95.3, 80.6)
- added REF**: Potentiometer_Bourns_3314J_Vertical, Potentiometer_SMD:Potentiometer_Bourns_3314J_Vertical, F.Cu at (65.3, 64.5)
- added REF**: Potentiometer_Bourns_3314G_Vertical, Potentiometer_SMD:Potentiometer_Bourns_3314G_Vertical, F.Cu at (53.0, 60.2)
