File: hardware/v2/pdlc.kicad_sch (KiCad schematic)
At the start: 58 parts, among them J1 TBP01R1-508-06BE, J3 SM04B-SRSS-TB, J6 Conn_ST_STDC14, J8 Conn_02x08_Odd_Even, Q1 MMBT3904, Q2 2N7002, U1 LP2985-33DBVR, U2 LM5158, U3 ISO1640, U4 STM32C051C8T6, U7 STM32L151C8T6A, U8 74LVC1G38

Commit message: Finalize for production of v2 revision.
Parts:
- removed C11, C12: 100n, Capacitor_SMD:C_0603_1608Metric, symbol Device:C
- removed J1: TBP01R1-508-06BE, TBP01R1-508-06BE:CUI_TBP01R1-508-06BE, symbol TBP01R1-508-06BE:TBP01R1-508-06BE
- removed J6: Conn_ST_STDC14, Samtec:SAMTEC_FTSH-107-01-L-DV-K-A, symbol Connector:Conn_ST_STDC14
- removed JP2: SolderJumper_2_Bridged, Jumper:SolderJumper-2_P1.3mm_Bridged_RoundedPad1.0x1.5mm, symbol Jumper:SolderJumper_2_Bridged
- removed R4: 2.2K, Resistor_SMD:R_0603_1608Metric, symbol Device:R
- removed U4: STM32C051C8T6, Package_QFP:LQFP-48_7x7mm_P0.5mm, symbol MCU_ST_STM32C0:STM32C031C6Tx
- removed U8: 74LVC1G38, symbol 74xGxx:74LVC1G38
- added C20, C21, C22, C23, C25, C26, C27, C28, C29: 100n, Capacitor_SMD:C_0402_1005Metric, symbol Device:C
- added C24: 1u, Capacitor_SMD:C_0603_1608Metric, symbol Device:C
- added D3, D4: PESD3V3L5UY, Package_TO_SOT_SMD:SOT-363_SC-70-6, symbol Power_Protection:PESD3V3L5UY
- added D5: LTST-C19HE1WT, LED_SMD:LED_LiteOn_LTST-C19HE1WT, symbol Device:LED_RGBA
- added D7: 1N5819WS, Diode_SMD:D_SOD-323, symbol Diode:1N5819WS
- added FB1: 450mOhm, Inductor_SMD:L_0603_1608Metric, symbol Device:FerriteBead_Small
- added J2: TBP04R12-500-04BE, Connector_Phoenix_MSTB:PhoenixContact_MSTBA_2,5_4-G_1x04_P5.00mm_Horizontal, symbol Connector_Generic:Conn_01x04
- added J5: Conn_ST_STDC14, Samtec:SAMTEC_FTSH-107-01-L-DV-K-A, symbol Connector:Conn_ST_STDC14
- added J6: TBP03R1-350-06BE, Connector_Phoenix_MC:PhoenixContact_MC_1,5_6-G-3.5_1x06_P3.50mm_Horizontal, symbol Connector_Generic:Conn_01x06
- added JP1: SolderJumper_2_Open, Jumper:SolderJumper-2_P1.3mm_Open_TrianglePad1.0x1.5mm, symbol Jumper:SolderJumper_2_Open
- added Q3: 2N7002, Package_TO_SOT_SMD:SOT-23, symbol Transistor_FET:2N7002
- added R12, R25, R26, R32: 470, Resistor_SMD:R_0402_1005Metric, symbol Device:R
- added R16, R27, R31: 2.2K, Resistor_SMD:R_0402_1005Metric, symbol Device:R
- added R17: 10K, Resistor_SMD:R_0402_1005Metric, symbol Device:R
- added R21, R33: 100K, Resistor_SMD:R_0402_1005Metric, symbol Device:R
- added R22, R29: 1K, Resistor_SMD:R_0402_1005Metric, symbol Device:R
- added R23, R24, R5, R6: 22K, Resistor_SMD:R_0402_1005Metric, symbol Device:R
- added SW1, SW2: SW_Push, Button_Switch_SMD:SW_SPST_TS-1088-xR020, symbol Switch:SW_Push
- added U3: SN74LVC1G08DCKR, Package_TO_SOT_SMD:SOT-353_SC-70-5, symbol 74xGxx:74LVC1G08
- C1: renamed from C2; footprint Capacitor_SMD:C_0603_1608Metric -> Capacitor_SMD:C_0402_1005Metric; LCSC C14663 -> C1525; Rating 50V, X7R -> 16V, X7R
- C12: renamed from C8; MPN CL31B104KCFNNNE -> (none); Part (none) -> CL31B104KCFNNNE
- C13: renamed from C9; Alternative GCM32DC72A475KE02L -> (none); MPN HMK325C7475KN-TE -> (none); Part (none) -> HMK325C7475KN-TE; Part Alternative (none) -> GCM32DC72A475KE02L
- C14: renamed from C13; Alternative GCM32DC72A475KE02L -> (none); MPN HMK325C7475KN-TE -> (none); Part (none) -> HMK325C7475KN-TE; Part Alternative (none) -> GCM32DC72A475KE02L
- C15: renamed from C19; FT Rotation Offset (none) -> 180; MPN 2201010609TR -> (none); Part (none) -> 2201010609TR
- C18: renamed from C16; footprint Capacitor_SMD:C_0603_1608Metric -> Capacitor_SMD:C_0402_1005Metric; LCSC C21122 -> C1532
- C19: renamed from C10; value 4.7u -> 10u; LCSC C19666 -> C19702; Rating 16V, X5R -> 10V, X5R
- C2: footprint Capacitor_SMD:C_0603_1608Metric -> Capacitor_SMD:C_0402_1005Metric; LCSC C14663 -> C1525; Rating 50V, X7R -> 16V, X7R
- C4: renamed from C5; footprint Capacitor_SMD:C_0603_1608Metric -> Capacitor_SMD:C_0402_1005Metric; LCSC C57112 -> C15195
- C6: renamed from C18; FT Rotation Offset (none) -> 180; MPN 2210250609R00 -> (none); Part (none) -> 2210250609R00
- C7: renamed from C17; MPN CL32B106KAJNNNE -> (none); Part (none) -> CL32B106KAJNNNE
- C8: MPN CL32B106KAJNNNE -> (none); Part (none) -> CL32B106KAJNNNE
- C9: renamed from C3; MPN CL32B106KAJNNNE -> (none); Part (none) -> CL32B106KAJNNNE
- D1: renamed from D3; Alternative SMF16A-E3-08 -> (none); FT Rotation Offset (none) -> 0; Part Alternative (none) -> SMF16A-E3-08
- D2: renamed from D5; FT Rotation Offset (none) -> 0
- D6: renamed from D4; footprint LED_SMD:LED_0603_1608Metric_Pad1.05x0.95mm_HandSolder -> LED_SMD:LED_0603_1608Metric; Label (none) -> POWER; Rating RED -> RED, 2.4V
- J1: renamed from J3; Alternative GT-A1002WRS-104SBT01 -> (none); LCSC Alternative (none) -> C41431904; LCSC_Alternative C41431904 -> (none); Label EXT QWIIC -> EXT I2C; Part Alternative (none) -> GT-A1002WRS-104SBT01
- J3: Alternative GT-A1002WRS-104SBT01 -> (none); LCSC Alternative (none) -> C41431904; LCSC_Alternative C41431904 -> (none); Label EXT QWIIC -> EXT I2C; Part Alternative (none) -> GT-A1002WRS-104SBT01
- L1: FT Rotation Offset (none) -> 270; MPN 7447714150 -> (none); Part (none) -> 7447714150
- R1, R2: footprint Resistor_SMD:R_0603_1608Metric -> Resistor_SMD:R_0402_1005Metric; LCSC C4190 -> C25879
- R15: renamed from R29; footprint Resistor_SMD:R_0603_1608Metric -> Resistor_SMD:R_0402_1005Metric; LCSC C4190 -> C25879
- R18, R19: value 100K -> 10K; footprint Resistor_SMD:R_0603_1608Metric -> Resistor_SMD:R_0402_1005Metric; LCSC C25803 -> C25744
- R20: value 10K -> 100K; LCSC C25744 -> C25741; Rating 50V, 1% -> (none)
- R28: value 330K -> 2.2K; footprint Resistor_SMD:R_0603_1608Metric -> Resistor_SMD:R_0402_1005Metric; LCSC C23137 -> C25879; Rating 75V, 1% -> (none)
- R30: value 2.2K -> 22K; footprint Resistor_SMD:R_0603_1608Metric -> Resistor_SMD:R_0402_1005Metric; LCSC C4190 -> C25768
- renumbered C1 to C10, C7 to C11, C14 to C16, C15 to C17, C4 to C3, C6 to C5, F2 to F1, J8 to J4, Q2 to Q1, Q1 to Q2, R8 to R10, R9 to R11, R10 to R13, R17 to R14, R5 to R3, R6 to R4, R16 to R7, R11 to R8, R7 to R9, U3 to U2, U2 to U4, U7 to U5
Connections:
- net +5V is gone; now on net +3.3V: J4.4 (Pin_4)
- net EXP_PA11 is gone; now on net EXP_PB7: J4.11 (Pin_11)
- net EXP_PA12 is gone; now on net EXP_PC13: J4.14 (Pin_14)
- net EXP_PA8 is gone; now on net EXP_PB6: J4.12 (Pin_12)
- net EXP_PB12 is gone; now on net EXP_PB15: J4.10 (Pin_10)
- net I2C_SCL is gone; now on net EXT_I2C_SCL: R2.2, U2.3 (SCL1)
- net I2C_SDA is gone; now on net EXT_I2C_SDA: R1.2, U2.2 (SDA1)
- net SWCLK/BOOT0 is gone; now on net BOOT0: J4.16 (Pin_16)
- net +12V: now also L1.2, J6.6 (Pin_6); no longer L1.1
- net +3.3V: now also D6.2 (A), R20.1, R30.1, U5.1 (VLCD), U5.24 (VDD), U5.36 (VDD), U5.48 (VDD), C20.1, C21.1, C22.1, C23.1, D5.4 (A), FB1.1, J5.3 (VCC), R16.2, R21.1, R23.1, R24.1, R6.1, U3.5 (VCC); no longer J4.6 (Pin_6), R18.1, R19.1, R20.2, R30.2
- net 12V_IN: now also J2.2 (Pin_2)
- net BUS_GND: now also J1.MP (MountPin), J3.MP (MountPin)
- net CONSOLE_RX: now also R20.2, U5.31 (PA10), D4.3 (K2), J5.13 (VCP_RX); no longer R18.2
- net CONSOLE_TX: now also U5.30 (PA9), D4.1 (K1), J5.14 (VCP_TX), R21.2; no longer R19.2
- net EXP_PA15: now also J4.9 (Pin_9), U5.38 (PA15); no longer J4.13 (Pin_13)
- net EXP_PB13: now also J4.8 (Pin_8), U5.26 (PB13); no longer J4.9 (Pin_9)
- net EXT_I2C_SCL: now also U5.45 (PB8)
- net EXT_I2C_SDA: now also U5.46 (PB9)
- net GND: now also R18.2, R19.2, U5.23 (VSS), U5.35 (VSS), U5.47 (VSS), U5.8 (VSSA), C20.2, C21.2, C22.2, C23.2, C24.2, C25.2, C26.2, C27.2, C28.2, C29.2, D3.1 (K1), D3.2 (A), D4.2 (A), D7.2 (A), J2.1 (Pin_1), J5.5 (GND), J5.7 (GND), J6.1 (Pin_1), J6.4 (Pin_4), JP1.1 (A), Q3.2 (S), R17.2, R33.1, R5.2, SW1.1, SW2.1, U3.3 (GND); no longer J4.5 (Pin_5)
- net HV: no longer R28.1
- net HV_EN: now also U5.40 (PB4), R12.1; no longer Q1.1 (G)
- net HV_PG: now also U5.41 (PB5), R6.2, U3.1; no longer R20.1
- net INT_I2C_SCL: now also J4.6 (Pin_6), U5.21 (PB10), R16.1; no longer J4.8 (Pin_8), R30.1
- net INT_I2C_SDA: now also J4.5 (Pin_5), U5.22 (PB11); no longer J4.7 (Pin_7)
- net PDLC_ADJ_A: now also U5.14 (PA4)
- net PDLC_ADJ_B: now also U5.15 (PA5)
- net PDLC_EN: now also U5.29 (PA8), R5.1, U3.2
- net PDLC_EN_DRV: now also U3.4; no longer R28.2
- net PDLC_OUT_A: now also J2.3 (Pin_3)
- net PDLC_OUT_B: now also J2.4 (Pin_4)
- net PDLC_PG_A: now also U5.3 (PC14)
- net PDLC_PG_B: now also U5.4 (PC15)
- net SWDIO: now also U5.34 (PA13), D3.4 (K3), J5.4 (JTMS/SWDIO)
- net ~{RESET}: now also U5.7 (NRST), C26.1, D3.3 (K2), J5.12 (~{RST})
- net ~{CTRL_MODE}: now reaches U5.10 (PA0)
- net ~{CTRL_MODE}: now also C29.1, R31.1
- net ~{CTRL_SET}: now reaches U5.11 (PA1)
- net ~{CTRL_SET}: now also C27.1, R27.1
- net ~{CTRL_EN}: now reaches U5.12 (PA2)
- net ~{CTRL_EN}: now also R28.1, C28.1
- net EXP_PA3: now reaches U5.13 (PA3)
- net EXP_PA3: now also J4.13 (Pin_13)
- net LED_STATUS_R: now reaches U5.16 (PA6)
- net LED_STATUS_R: now also R22.2
- net LED_STATUS_G: now reaches U5.17 (PA7)
- net LED_STATUS_G: now also R25.1
- net LED_STATUS_B: now reaches U5.18 (PB0)
- net LED_STATUS_B: now also R26.1
- net LED_POWER: now reaches U5.19 (PB1)
- net LED_POWER: now also R29.2
- net EXP_PC13: now reaches U5.2 (PC13)
- net EXP_PC13: now also R19.1
- net BOOT1: now reaches U5.20 (PB2)
- net BOOT1: now also R18.1
- net LOAD_EN: now reaches U5.25 (PB12)
- net LOAD_EN: now also R32.1, R33.2
- net EXP_PB14: now reaches U5.27 (PB14)
- net EXP_PB14: now also J4.7 (Pin_7)
- net EXP_PB15: now reaches U5.28 (PB15)
- net SWCLK: now reaches U5.37 (PA14)
- net SWCLK: now also D3.5 (K4), J5.6 (JCLK/SWCLK)
- net SWO: now reaches U5.39 (PB3)
- net SWO: now also D3.6 (K5), J5.8 (JTDO/SWO)
- net EXP_PB6: now reaches U5.42 (PB6)
- net EXP_PB7: now reaches U5.43 (PB7)
- net BOOT0: now reaches U5.44 (BOOT0)
- net BOOT0: now also R17.1
- net VDDA: now reaches U5.9 (VDDA)
- net VDDA: now also C24.1, C25.1, FB1.2
- net at D6.1 (K): now also R29.1
- net at D2.2 (A), U4.13 (SW), U4.14 (SW): now also L1.1; no longer L1.2
- new net: D5.1 (RK), R22.1
- new net: D5.2 (GK), R25.2
- new net: D5.3 (BK), R26.2
- new net: Q1.1 (G), R12.2
- new net: Q3.1 (G), R32.2
- new net LOAD_OUT: D7.1 (K), J6.5 (Pin_5), Q3.3 (D)
- new net ~{CTRL_EN_IN}: D4.6 (K5), J6.2 (Pin_2), JP1.2 (B), R24.2, R28.2
- new net ~{CTRL_MODE_IN}: D4.5 (K4), J6.3 (Pin_3), R30.2, R31.2, SW2.2
- new net ~{CTRL_SET_IN}: D4.4 (K3), R23.2, R27.2, SW1.2
- no-connect marks 6 -> 7
Other:
- note added: "CONTROL I/O"
- note added: "Circuit protection for power input: - Internal: 2 A polyfuse, reverse polarity, overvoltage - External: 3 A fuse, 20 AWG minimum recommended Pin 1: Power input, ground Pin 2: Power input, 12 V DC nominal, 16 V DC maximum Pin 3/4: PDLC output A/B, 60 V AC (peak-to-peak) nominal"
- note added: "Datasheet: In STM32L151xxxxA devices VLCD should be connected to VDD"
- note added: "EXTERNAL I2C INTERFACE (QWIIC)"
- note added: "HSE"
- note added: "INDICATORS"
- note added: "Load output rated for 200 mA at 20 V, sufficient for an indicator, optocoupler, or small relay coil The SET button cannot be wired remotely because its function requires the indicators to be visible ESD protection on all switch inputs"
- note added: "Outputs 300 mA between the terminals at 60 V AC RMS The drivers remain off unless HV_PG and PDLC_EN are both high (for functional safety) and thereby ensures that VIN > 3.3 so UVLO/EN remains below VIN + 0.3 V as required by the IC"
- note added: "POWER TERMINAL BLOCK"
- note added: "Programmed via SWD with STLINK-V3 and an STDC14 cable Can also access the system bootloader over UART by pulling BOOT0 high during RESET Unused pins are exposed via an expansion port including an internal I2C interface"
- note added: "STM32L151C8T6 MICROCONTROLLER"
- note added: "USB"
- note added: "VDD"
- note added: "VDDA"
- note removed: "Circuit protection for power input: - Internal: 2 A polyfuse, reverse polarity, overvoltage - External: 3 A fuse, 20 AWG minimum recommended Pin 1: Power ground Pin 2: Power input, 12 V DC nominal, 16 V DC maximum Pin 3: ENABLE switch input, active low Pin 4: MODE switch input, active low Pin 5/6: PDLC output A/B, 60 V AC (peak-to-peak) nominal"
- note removed: "EXTERNAL QWIIC INTERFACE"
- note removed: "INDICATOR"
- note removed: "Outputs 300 mA between the terminals at 60 V AC RMS The drivers remain off unless HV_PG and PDLC_EN are both high and ensures that the voltage at UVLO/EN remains below VIN + 0.3 V as required by the IC"
- note removed: "Programmed via SWD with STLINK-V3 and an STDC14 cable Can also access the system bootloader over I2C or UART by pulling BOOT0 low during RESET Unused pins are exposed via an expansion port including an internal I2C port"
- note removed: "STM32C051 MICROCONTROLLER"
- note removed: "Steady on when the PDLC film is switched on Flashing when a fault occurs"
- note removed: "TERMINAL BLOCK"
- moved on the sheet: C1, C19, D1, D6, F1, J1, J3, J4, L1, Q1, Q2, R1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
