File: hardware/v2/pdlc.kicad_sch (KiCad schematic)
At the start: 58 parts, among them J1 TBP01R1-508-06BE, J3 SM04B-SRSS-TB, J6 Conn_ST_STDC14, J8 Conn_02x08_Odd_Even, Q1 MMBT3904, Q2 2N7002, U1 LP2985-33DBVR, U2 LM5158, U3 ISO1640, U4 STM32C051C8T6, U7 STM32L151C8T6A, U8 74LVC1G38

Commit message: WIP
Parts:
- removed C11: 100n, Capacitor_SMD:C_0603_1608Metric, symbol Device:C
- removed J1: TBP01R1-508-06BE, TBP01R1-508-06BE:CUI_TBP01R1-508-06BE, symbol TBP01R1-508-06BE:TBP01R1-508-06BE
- removed J6: Conn_ST_STDC14, Samtec:SAMTEC_FTSH-107-01-L-DV-K-A, symbol Connector:Conn_ST_STDC14
- removed JP2: SolderJumper_2_Bridged, Jumper:SolderJumper-2_P1.3mm_Bridged_RoundedPad1.0x1.5mm, symbol Jumper:SolderJumper_2_Bridged
- removed R30: 2.2K, Resistor_SMD:R_0603_1608Metric, symbol Device:R
- removed U4: STM32C051C8T6, Package_QFP:LQFP-48_7x7mm_P0.5mm, symbol MCU_ST_STM32C0:STM32C031C6Tx
- added C20, C21, C22, C23, C25, C27, C28, C29: 100n, Capacitor_SMD:C_0402_1005Metric, symbol Device:C
- added C24: 1u, Capacitor_SMD:C_0603_1608Metric, symbol Device:C
- added D3, D4: PESD3V3L5UY, Package_TO_SOT_SMD:SOT-363_SC-70-6, symbol Power_Protection:PESD3V3L5UY
- added D6: 1N5819WS, Diode_SMD:D_SOD-323, symbol Diode:1N5819WS
- added FB1: 450mOhm, Inductor_SMD:L_0603_1608Metric, symbol Device:FerriteBead_Small
- added J2: TBP04R12-500-04BE, Connector_Phoenix_MSTB:PhoenixContact_MSTBA_2,5_4-G_1x04_P5.00mm_Horizontal, symbol Connector_Generic:Conn_01x04
- added J4: BM04B-SRSS-TB, Connector_JST:JST_SH_BM04B-SRSS-TB_1x04-1MP_P1.00mm_Vertical, symbol Connector_Generic_MountingPin:Conn_01x04_MountingPin
- added J5: Conn_ST_STDC14, Samtec:SAMTEC_FTSH-107-01-L-DV-K-A, symbol Connector:Conn_ST_STDC14
- added J7: TBP03R1-350-06BE, Connector_Phoenix_MC:PhoenixContact_MC_1,5_6-G-3.5_1x06_P3.50mm_Horizontal, symbol Connector_Generic:Conn_01x06
- added JP1: SolderJumper_2_Open, Jumper:SolderJumper-2_P1.3mm_Open_TrianglePad1.0x1.5mm, symbol Jumper:SolderJumper_2_Open
- added Q3: 2N7002, Package_TO_SOT_SMD:SOT-23, symbol Transistor_FET:2N7002
- added R12, R28: 470, Resistor_SMD:R_0402_1005Metric, symbol Device:R
- added R16, R24, R25, R27: 2.2K, Resistor_SMD:R_0402_1005Metric, symbol Device:R
- added R17: 10K, Resistor_SMD:R_0402_1005Metric, symbol Device:R
- added R20, R29: 100K, Resistor_SMD:R_0402_1005Metric, symbol Device:R
- added R22, R23, R26: 22K, Resistor_SMD:R_0402_1005Metric, symbol Device:R
- added SW1, SW2: SW_Push, symbol Switch:SW_Push
- C1: renamed from C2; footprint Capacitor_SMD:C_0603_1608Metric -> Capacitor_SMD:C_0402_1005Metric; LCSC C14663 -> C1525; Rating 50V, X7R -> 16V, X7R
- C19: renamed from C10; value 4.7u -> 10u; LCSC C19666 -> C19702; Rating 16V, X5R -> 10V, X5R
- C2: footprint Capacitor_SMD:C_0603_1608Metric -> Capacitor_SMD:C_0402_1005Metric; LCSC C14663 -> C1525; Rating 50V, X7R -> 16V, X7R
- C4: renamed from C5; footprint Capacitor_SMD:C_0603_1608Metric -> Capacitor_SMD:C_0402_1005Metric; LCSC C57112 -> C15195
- J1: renamed from J3; Label EXT QWIIC -> EXT I2C
- J3: Label EXT QWIIC -> EXT I2C
- R1, R2: footprint Resistor_SMD:R_0603_1608Metric -> Resistor_SMD:R_0402_1005Metric; LCSC C4190 -> C25879
- R15: renamed from R29; footprint Resistor_SMD:R_0603_1608Metric -> Resistor_SMD:R_0402_1005Metric; LCSC C4190 -> C25879
- R18: value 100K -> 10K; footprint Resistor_SMD:R_0603_1608Metric -> Resistor_SMD:R_0402_1005Metric; LCSC C25803 -> C25744
- R19: footprint Resistor_SMD:R_0603_1608Metric -> Resistor_SMD:R_0402_1005Metric; LCSC C25803 -> C25741
- R6: renamed from R20; Rating 50V, 1% -> 50V
- renumbered C1 to C10, C7 to C11, C8 to C12, C9 to C13, C13 to C14, C19 to C15, C14 to C16, C15 to C17, C16 to C18, C12 to C26, C4 to C3, C6 to C5, C18 to C6, C17 to C7, C3 to C9, D3 to D1, D5 to D2, D4 to D5, F2 to F1, J8 to J6, Q2 to Q1, Q1 to Q2, R8 to R10, R9 to R11, R10 to R13, R17 to R14, R4 to R21, R28 to R3, R5 to R4, R6 to R5, R16 to R7, R11 to R8, R7 to R9, U3 to U2, U8 to U3, U2 to U4, U7 to U5
Connections:
- net I2C_SCL is gone; now on net EXT_I2C_SCL: R2.2, U2.3 (SCL1)
- net I2C_SDA is gone; now on net EXT_I2C_SDA: R1.2, U2.2 (SDA1)
- net STATUS is gone; now on net LED_AUX: R21.2
- net SWCLK/BOOT0 is gone; now on net BOOT0: J6.16 (Pin_16)
- net +12V: now also J7.6 (Pin_6)
- net +3.3V: now also D5.2 (A), U5.1 (VLCD), U5.24 (VDD), U5.36 (VDD), U5.48 (VDD), C20.1, C21.1, C22.1, C23.1, FB1.1, J4.2 (Pin_2), J5.3 (VCC), R16.2, R20.1, R22.1, R23.1, R26.1; no longer R18.1
- net 12V_IN: now also J2.2 (Pin_2)
- net CONSOLE_RX: now also R19.2, D3.3 (K2), J5.13 (VCP_RX); no longer R18.2
- net CONSOLE_TX: now also D3.1 (K1), J5.14 (VCP_TX), R20.2; no longer R19.2
- net EXT_I2C_SCL: now also U5.45 (PB8)
- net EXT_I2C_SDA: now also U5.46 (PB9)
- net GND: now also R18.2, U5.23 (VSS), U5.35 (VSS), U5.47 (VSS), U5.8 (VSSA), C20.2, C21.2, C22.2, C23.2, C24.2, C25.2, C27.2, C28.2, C29.2, D3.2 (A), D4.2 (A), D6.2 (A), J2.1 (Pin_1), J4.1 (Pin_1), J5.5 (GND), J5.7 (GND), J7.1 (Pin_1), J7.4 (Pin_4), JP1.1 (A), Q3.2 (S), R17.2, R29.1, SW1.1, SW2.1
- net HV_EN: now also R12.1; no longer Q1.1 (G)
- net INT_I2C_SCL: now also U5.21 (PB10), J4.4 (Pin_4), R16.1
- net INT_I2C_SDA: now also U5.22 (PB11), J4.3 (Pin_3)
- net PDLC_ADJ_A: now also U5.14 (PA4)
- net PDLC_ADJ_B: now also U5.15 (PA5)
- net PDLC_OUT_A: now also J2.3 (Pin_3)
- net PDLC_OUT_B: now also J2.4 (Pin_4)
- net SWDIO: now also U5.34 (PA13), D3.4 (K3), J5.4 (JTMS/SWDIO)
- net ~{RESET}: now also U5.7 (NRST), D3.6 (K5), J5.12 (~{RST})
- net ~{CTRL_MODE}: now reaches U5.10 (PA0)
- net ~{CTRL_MODE}: now also C29.1, R27.1
- net ~{CTRL_SET}: now reaches U5.11 (PA1)
- net ~{CTRL_SET}: now also C27.1, R24.1
- net LED_STATUS_R: now reaches U5.16 (PA6)
- net LED_STATUS_G: now reaches U5.17 (PA7)
- net LED_STATUS_G: now also U5.18 (PB0)
- net LED_AUX: now reaches U5.19 (PB1)
- net ~{CTRL_ENABLE}: now reaches U5.2 (PC13)
- net ~{CTRL_ENABLE}: now also C28.1, R25.1
- net BOOT1: now reaches U5.20 (PB2)
- net BOOT1: now also R18.1
- net LOAD_EN: now reaches U5.25 (PB12)
- net LOAD_EN: now also R28.1, R29.2
- net SWCLK: now reaches U5.37 (PA14)
- net SWCLK: now also D3.5 (K4), J5.6 (JCLK/SWCLK)
- net SWO: now reaches U5.39 (PB3)
- net SWO: now also D4.1 (K1), J5.8 (JTDO/SWO)
- net BOOT0: now reaches U5.44 (BOOT0)
- net BOOT0: now also D4.6 (K5), R17.1
- net VDDA: now reaches U5.9 (VDDA)
- net VDDA: now also C24.1, C25.1, FB1.2
- new net: D4.4 (K3), R22.2, R24.2, SW1.2
- new net: Q1.1 (G), R12.2
- new net: Q3.1 (G), R28.2
- new net LOAD: D6.1 (K), J7.5 (Pin_5), Q3.3 (D)
- new net ~{CTRL_ENABLE_IN}: D4.5 (K4), J7.2 (Pin_2), JP1.2 (B), R23.2, R25.2
- new net ~{CTRL_MODE_IN}: D4.3 (K2), J7.3 (Pin_3), R26.2, R27.2, SW2.2
- no-connect marks 6 -> 8
Other:
- note added: "CONTROL I/O"
- note added: "Circuit protection for power input: - Internal: 2 A polyfuse, reverse polarity, overvoltage - External: 3 A fuse, 20 AWG minimum recommended Pin 1: Power input, ground Pin 2: Power input, 12 V DC nominal, 16 V DC maximum Pin 3/4: PDLC output A/B, 60 V AC (peak-to-peak) nominal"
- note added: "Datasheet: In STM32L151xxxxA devices VLCD should be connected to VDD"
- note added: "EXTERNAL I2C INTERFACE (QWIIC)"
- note added: "INDICATORS"
- note added: "Load output rated for 200 mA at 20 V, sufficient for an indicator, optocoupler, or small relay coil The SET button cannot be wired remotely because its function requires the indicators to be visible ESD protection on all switch inputs"
- note added: "Outputs 300 mA between the terminals at 60 V AC RMS The drivers remain off unless HV_PG and PDLC_EN are both high (for functional safety) and ensures that the voltage at UVLO/EN remains below VIN + 0.3 V as required by the IC"
- note added: "POWER TERMINAL BLOCK"
- note added: "Programmed via SWD with STLINK-V3 and an STDC14 cable Can also access the system bootloader over UART by pulling BOOT0 low during RESET Unused pins are exposed via an expansion port including an internal I2C interface (QWIIC)"
- note added: "STM32L151C8T6 MICROCONTROLLER"
- note added: "VDD"
- note added: "VDDA"
- note removed: "Circuit protection for power input: - Internal: 2 A polyfuse, reverse polarity, overvoltage - External: 3 A fuse, 20 AWG minimum recommended Pin 1: Power ground Pin 2: Power input, 12 V DC nominal, 16 V DC maximum Pin 3: ENABLE switch input, active low Pin 4: MODE switch input, active low Pin 5/6: PDLC output A/B, 60 V AC (peak-to-peak) nominal"
- note removed: "EXTERNAL QWIIC INTERFACE"
- note removed: "INDICATOR"
- note removed: "Outputs 300 mA between the terminals at 60 V AC RMS The drivers remain off unless HV_PG and PDLC_EN are both high and ensures that the voltage at UVLO/EN remains below VIN + 0.3 V as required by the IC"
- note removed: "Programmed via SWD with STLINK-V3 and an STDC14 cable Can also access the system bootloader over I2C or UART by pulling BOOT0 low during RESET Unused pins are exposed via an expansion port including an internal I2C port"
- note removed: "STM32C051 MICROCONTROLLER"
- note removed: "Steady on when the PDLC film is switched on Flashing when a fault occurs"
- note removed: "TERMINAL BLOCK"
- moved on the sheet: C1, C19, C26, D1, D5, F1, J1, J3, J6, Q1, Q2, R1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
